File: RgbwLedDriver.brd (EAGLE design)
At the start: 75 x 35 mm, 47 parts, among them CN1 LED1, CN2 LED2, CN3 LED3, CN4 LED4, CN5 POWER, CN6 I2C, CN7 POWER, CN8 I2C, IC1 PCA9685BS, J1 A0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

Commit message: 電源のシンボルを変更
Connections:
- net +3V renamed +3.3V
- net +7.2V renamed +7.4V
Changed lines of the file:
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@@
 <wire x1="70" y1="22" x2="69" y2="22" width="0.2" layer="16"/>
 </signal>
-<signal name="+3V">
+<signal name="+3.3V">
 <contactref element="IC1" pad="25"/>
 <contactref element="RN1" pad="7"/>
@@
 <wire x1="19.5" y1="8" x2="17.5" y2="6" width="0.2" layer="1"/>
 </signal>
-<signal name="+7.2V">
-<contactref element="CN5" pad="1"/>
-<contactref element="CN7" pad="1"/>
+<signal name="+7.4V">
 <contactref element="CN1" pad="1"/>
-<contactref element="CN2" pad="1"/>
-<contactref element="CN4" pad="1"/>
-<contactref element="CN3" pad="1"/>
 <polygon width="0.2" layer="16" thermals="no">
 <vertex x="20.5" y="28"/>
@@
 <vertex x="23.5" y="28"/>
 </polygon>
+<contactref element="CN2" pad="1"/>
+<contactref element="CN3" pad="1"/>
+<contactref element="CN4" pad="1"/>
+<contactref element="CN5" pad="1"/>
+<contactref element="CN7" pad="1"/>
 </signal>
 </signals>
